File: Hardware/C4V1/C4V1.sch (KiCad schematic (older format))
At the start: 27 parts, among them IC1 W25Q16JVSNIQ, IC2 MB85RS256TYPNF-G-AWERE2, J1 48037-2100, J2 Prawo, J3 Lewo, U1 LDLN050PU33, U2 ESDALCL6-2SC6, U3 STM32G4A1KEU6, Y1 ECS-80-8-33Q-ADS-TR3

Commit message: Przedostatnie poprawki
Parts:
- removed J2: Prawo, Connector_PinHeader_2.54mm:PinHeader_1x20_P2.54mm_Vertical, symbol Connector:Conn_01x20_Male
- removed J3: Lewo, Connector_PinHeader_2.54mm:PinHeader_1x20_P2.54mm_Vertical, symbol Connector:Conn_01x20_Male
- added C12, C13, C14, C15, C16, C17: 100n/X5R/10V, Capacitor_SMD:C_0402_1005Metric, symbol Device:C
- added D1: LED, LED_SMD:LED_0603_1608Metric, symbol Device:LED
- added J2: Conn_01x08_Male, Connector_PinHeader_2.54mm:PinHeader_1x08_P2.54mm_Vertical, symbol Connector:Conn_01x08_Male
- added J3: Conn_01x05_Female, C4V1:Programator, symbol Connector:Conn_01x05_Female
- added R10, R11, R12, R8, R9: 10k/5%/0.1W, Resistor_SMD:R_0402_1005Metric, symbol Device:R
- added R7: /5%/0.1W, Resistor_SMD:R_0402_1005Metric, symbol Device:R
- added SW1, SW2, SW3, SW4, SW5, SW6, SW7: SW_Push, Button_Switch_SMD:SW_Push_1P1T_NO_6x6mm_H9.5mm, symbol Switch:SW_Push
- C1, C10, C11, C2, C3, C4, C5, C6, C8, C9: footprint Capacitor_SMD:C_0603_1608Metric -> Capacitor_SMD:C_0402_1005Metric
- R1, R2, R3, R4, R5, R6: footprint Resistor_SMD:R_0603_1608Metric -> Resistor_SMD:R_0402_1005Metric
Connections:
- net FLASH_CS is gone; now on net ~FLASH_CS: IC1.1 (~CS)
- net FRAM_CS is gone; now on net ~FRAM_CS: IC2.1 (~CS)
- net X is gone; now on net DOWN: U3.28 (PB5)
- net Y is gone; now on net RIGHT: U3.30 (PB7)
- net +3V3: now also C17.2, J2.8 (Pin_8), J3.1 (Pin_1), R10.1, R11.1, R12.1, R8.1, R9.1, SW6.1
- net CLK: now also J2.4 (Pin_4)
- net DOWN: now also C15.1, R11.2, SW2.1; no longer U3.27 (PB4)
- net GND: now also C12.2, C13.2, C14.2, C15.2, C16.2, D1.1 (K), J2.7 (Pin_7), J3.2 (Pin_2), SW1.2, SW2.2, SW3.2, SW4.2, SW5.2, SW7.1
- net LEFT: now also U3.27 (PB4), C14.1, R10.2, SW3.1
- net MOSI: now also J2.5 (Pin_5)
- net RIGHT: now also C13.1, R9.2, SW4.1; no longer U3.29 (PB6)
- net UP: now also U3.26 (PB3), C16.1, R12.2, SW1.1
- net ~FLASH_CS: now reaches U3.19 (PA9)
- net ~FRAM_CS: now reaches U3.20 (PA10)
- net SWDIO: now reaches U3.23 (PA13)
- net SWDIO: now also J3.5 (Pin_5)
- net SWCLK: now reaches U3.24 (PA14)
- net SWCLK: now also J3.4 (Pin_4)
- net at U3.25 (PA15): now also R7.2
- net BOOT0: now reaches R6.1, U3.31 (PB8-BOOT0)
- net BOOT0: now also C17.1, SW6.2
- net RST_SWD: now reaches C8.1, R5.2, U3.4 (PG10-NRST)
- net RST_SWD: now also J3.3 (Pin_3), SW7.2
- net ~RES: now reaches U3.5 (PA0)
- net ~RES: now also J2.1 (Pin_1)
- net DC: now reaches U3.7 (PA2)
- net DC: now also J2.2 (Pin_2)
- net ~CS: now reaches U3.8 (PA3)
- net ~CS: now also J2.3 (Pin_3)
- new net: D1.2 (A), R7.1
- new net OK: C12.1, R8.2, SW5.1, U3.29 (PB6)
- no-connect marks 17 -> 1
Other:
- moved on the sheet: IC2, R3, R4, R6

Commit message: Dodano początkową konfiguracje
Connections:
- net +3V3: no longer C17.2
- net GND: now also C17.2
Changed lines of the file:
@@
 	2450 2000 2450 2050
 Connection ~ 2450 2050
-Wire Wire Line
-	2450 2350 1650 2350
-Wire Wire Line
-	1650 2350 1650 2100
 $Comp
-L power:+3.3V #PWR0146
-U 1 1 6434ABF1
-P 1650 2100
-F 0 "#PWR0146" H 1650 1950 50  0001 C CNN
-F 1 "+3.3V" H 1665 2273 50  0000 C CNN
-F 2 "" H 1650 2100 50  0001 C CNN
-F 3 "" H 1650 2100 50  0001 C CNN
-	1    1650 2100
+L power:GND #PWR?
+U 1 1 644403F8
+P 2450 2350
+F 0 "#PWR?" H 2450 2100 50  0001 C CNN
+F 1 "GND" H 2455 2177 50  0000 C CNN
+F 2 "" H 2450 2350 50  0001 C CNN
+F 3 "" H 2450 2350 50  0001 C CNN
+	1    2450 2350
 	1    0    0    -1
 $EndComp
