File: Hardware/C4V1/_autosave-C4V1.kicad_pcb (KiCad board)
At the start: 2 copper layers, 70 x 40 mm, 47 parts, among them IC1 W25Q16JVSNIQ, IC2 MB85RS256TYPNF-G-AWERE2, J1 48037-2100, J2 Conn_01x08_Male, J3 Conn_01x05_Female, SW1 SW_Push, SW2 SW_Push, SW3 SW_Push, SW4 SW_Push, SW5 SW_Push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

Commit message: Przedostatnie poprawki
Changed lines of the file:
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@@
     (thickness 1.6)
     (drawings 22)
-    (tracks 526)
+    (tracks 524)
     (zones 0)
     (modules 47)
@@
     (34 B.Paste user)
     (35 F.Paste user)
-    (36 B.SilkS user hide)
+    (36 B.SilkS user)
     (37 F.SilkS user)
     (38 B.Mask user)
@@
     (tags LED)
     (attr smd)
-    (fp_text reference D1 (at 0 1.43) (layer B.SilkS)
+    (fp_text reference D1 (at -2.61 -0.02) (layer B.SilkS)
       (effects (font (size 1 1) (thickness 0.15)) (justify mirror))
     )
@@
   (segment (start 111.02 119.28) (end 109.58 119.28) (width 0.25) (layer F.Cu) (net 3))
   (segment (start 112.2 119.28) (end 111.12 119.28) (width 0.25) (layer F.Cu) (net 3))
-  (segment (start 100.700001 111.000001) (end 100 110.3) (width 0.25) (layer F.Cu) (net 3))
-  (segment (start 100.700001 112.400001) (end 100.700001 111.000001) (width 0.25) (layer F.Cu) (net 3))
-  (segment (start 100.75 112.45) (end 100.700001 112.400001) (width 0.25) (layer F.Cu) (net 3))
-  (segment (start 100.75 112.75) (end 100.75 112.45) (width 0.25) (layer F.Cu) (net 3))
   (segment (start 100 110.3) (end 100 110.3) (width 0.25) (layer F.Cu) (net 3))
   (via (at 100 110.3) (size 0.8) (drill 0.4) (layers F.Cu B.Cu) (net 3))
@@
   (via (at 114.66 110.27) (size 0.8) (drill 0.4) (layers F.Cu B.Cu) (net 3))
   (via (at 115.42 110.98) (size 0.8) (drill 0.4) (layers F.Cu B.Cu) (net 3))
+  (segment (start 100.75 111.05) (end 100 110.3) (width 0.25) (layer F.Cu) (net 3))
+  (segment (start 100.75 112.75) (end 100.75 111.05) (width 0.25) (layer F.Cu) (net 3))
   (segment (start 107.422626 119.525) (end 107.95 119.525) (width 0.25) (layer F.Cu) (net 4))
   (segment (start 107.299999 119.647627) (end 107.422626 119.525) (width 0.25) (layer F.Cu) (net 4))

Commit message: Dodano początkową konfiguracje
Parts:
- D1: value LED -> WS2812B; footprint LED_SMD:LED_0603_1608Metric -> LED_SMD:LED_WS2812B_PLCC4_5.0x5.0mm_P3.2mm; moved to F.Cu
- moved D1 5.08 mm to (107.1, 101.5), turned to 90 degrees
Connections:
- C17 pad 2: +3V3 -> GND
- D1 pad 1: GND -> VBUS
- J3 pad 1: +3V3 -> VBUS
- R7 pad 1: Net-(D1-Pad2) -> Net-(D1-Pad4)
Routing:
- net VBUS: track 18.4 -> 162.5 mm, vias 0 -> 2
- net Net-(D1-Pad2): track 9.42 -> 0.00 mm, vias 1 -> 0
- net Net-(D1-Pad4): track 0.00 -> 7.79 mm
- net +3V3: track 223.8 -> 217.5 mm, vias 12 -> 11
- net MOSI: track 32.2 -> 31.4 mm
- net GND: vias 109 -> 116
