File: Hardware/C4V1/_autosave-C4V1.sch (KiCad schematic (older format))
At the start: 47 parts, among them IC1 W25Q16JVSNIQ, IC2 MB85RS256TYPNF-G-AWERE2, J1 48037-2100, J2 Conn_01x08_Male, J3 Conn_01x05_Female, SW1 SW_Push, SW2 SW_Push, SW3 SW_Push, SW4 SW_Push, SW5 SW_Push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

Commit message: Dodano początkowe struktury
Parts:
- removed D1: WS2812B, LED_SMD:LED_WS2812B_PLCC4_5.0x5.0mm_P3.2mm, symbol LED:WS2812B
- added D1: LED, LED_SMD:LED_0603_1608Metric, symbol Device:LED
Connections:
- wire segments 142 -> 145
- no-connect marks 2 -> 1
Changed lines of the file:
@@
 OK
+$Comp
+L Device:LED D1
+U 1 1 6418BE45
+P 4200 1400
+F 0 "D1" V 4147 1480 50  0000 L CNN
+F 1 "LED" V 4238 1480 50  0000 L CNN
+F 2 "LED_SMD:LED_0603_1608Metric" H 4200 1400 50  0001 C CNN
+F 3 "~" H 4200 1400 50  0001 C CNN
+	1    4200 1400
+	0    1    1    0
+$EndComp
 $Comp
 L Device:R R7
@@
 	5150 2150 5150 1950
 $Comp
+L power:+3.3V #PWR0124
+U 1 1 642BA314
+P 5150 1950
+F 0 "#PWR0124" H 5150 1800 50  0001 C CNN
+F 1 "+3.3V" H 5165 2123 50  0000 C CNN
+F 2 "" H 5150 1950 50  0001 C CNN
+F 3 "" H 5150 1950 50  0001 C CNN
+	1    5150 1950
+	1    0    0    -1
+$EndComp
+Wire Wire Line
+	4200 1250 4200 1100
+Wire Wire Line
+	4200 1100 4500 1100
+Wire Wire Line
+	4500 1100 4500 1350
+$Comp
 L power:GND #PWR0125
 U 1 1 642C48E7
-P 4500 1250
-F 0 "#PWR0125" H 4500 1000 50  0001 C CNN
-F 1 "GND" H 4505 1077 50  0000 C CNN
-F 2 "" H 4500 1250 50  0001 C CNN
-F 3 "" H 4500 1250 50  0001 C CNN
-	1    4500 1250
+P 4500 1350
+F 0 "#PWR0125" H 4500 1100 50  0001 C CNN
+F 1 "GND" H 4505 1177 50  0000 C CNN
+F 2 "" H 4500 1350 50  0001 C CNN
+F 3 "" H 4500 1350 50  0001 C CNN
+	1    4500 1350
 	1    0    0    -1
 $EndComp
@@
 Connection ~ 2450 2050
 $Comp
-L power:GND #PWR0146
+L power:GND #PWR?
 U 1 1 644403F8
 P 2450 2350
-F 0 "#PWR0146" H 2450 2100 50  0001 C CNN
+F 0 "#PWR?" H 2450 2100 50  0001 C CNN
 F 1 "GND" H 2455 2177 50  0000 C CNN
 F 2 "" H 2450 2350 50  0001 C CNN
@@
 	1    0    0    -1
 $EndComp
-$Comp
-L power:VBUS #PWR0124
-U 1 1 64452E1F
-P 5150 1950
-F 0 "#PWR0124" H 5150 1800 50  0001 C CNN
-F 1 "VBUS" H 5165 2123 50  0000 C CNN
-F 2 "" H 5150 1950 50  0001 C CNN
-F 3 "" H 5150 1950 50  0001 C CNN
-	1    5150 1950
-	1    0    0    -1
-$EndComp
-$Comp
-L LED:WS2812B D1
-U 1 1 6446E2A2
-P 4200 1250
-F 0 "D1" V 4246 906 50  0000 R CNN
-F 1 "WS2812B" V 4155 906 50  0000 R CNN
-F 2 "LED_SMD:LED_WS2812B_PLCC4_5.0x5.0mm_P3.2mm" H 4250 950 50  0001 L TNN
-F 3 "https://cdn-shop.adafruit.com/datasheets/WS2812B.pdf" H 4300 875 50  0001 L TNN
-	1    4200 1250
-	0    -1   -1   0
-$EndComp
-$Comp
-L power:VBUS #PWR0147
-U 1 1 644A9E3F
-P 3900 1250
-F 0 "#PWR0147" H 3900 1100 50  0001 C CNN
-F 1 "VBUS" H 3915 1423 50  0000 C CNN
-F 2 "" H 3900 1250 50  0001 C CNN
-F 3 "" H 3900 1250 50  0001 C CNN
-	1    3900 1250
-	1    0    0    -1
-$EndComp
-NoConn ~ 4200 950
 $EndSCHEMATC
